File: HW/REV2/KicadV2/xyp-gpib.kicad_pcb (KiCad board)
At the start: 2 copper layers, 54 x 15 mm, 25 parts, among them J1 USB_C_Receptacle_USB2.0, SW1 SW_Push, U1 ATmega32U4-MU, Y1 CX2016DB16000D0WZRC1

Commit message: commit
Parts:
- added G***: LOGO, LOGO, B.Cu at (187.7, 82.6)
- GPIB1: value 112-024-113R001 -> 111-024-113L001
- R7: value 10k -> 5k1
Connections:
- net /D+ renamed /Da+
- net /D- renamed /Da-
- net Net-(U1-D+) renamed /Db-
- net Net-(U1-D-) renamed /Db+
Routing:
- net +5V: track 94.8 -> 14.5 mm, vias 4 -> 13
- net GND: track 32.4 -> 45.1 mm, vias 45 -> 27
- net /DIO4: track 51.8 -> 39.1 mm, vias 2 -> 1
- net /IFC: track 21.0 -> 14.5 mm
- net /DIO1: track 44.6 -> 38.1 mm, vias 2 -> 1
- net /DIO2: track 41.0 -> 35.8 mm, vias 2 -> 1
- net /MISO: track 16.2 -> 12.1 mm
- net /NRFD: track 27.1 -> 24.2 mm
- net /DIO6: track 37.5 -> 34.9 mm
- net /MOSI: track 60.1 -> 58.2 mm, vias 2 -> 3
- net /SCK: track 18.0 -> 16.4 mm, vias 0 -> 2
- net /ATN: track 8.89 -> 10.3 mm
- net /Da-: track 30.2 -> 29.1 mm
- net /REN: track 23.1 -> 24.1 mm
- net /DIO8: track 26.8 -> 27.8 mm
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- added copper zone on B.Cu, net +5V
- added copper zone on F.Cu, net +5V
- added copper zone on In1.Cu, net GND
- added copper zone on In2.Cu, net GND
- removed copper zone on B.Cu, net GND
- removed copper zone on F.Cu, net GND
Other:
- copper layers 2 -> 4
- board text added: "REV 2.1"
- board text removed: "REV 2"
