File: HW/REV2/KicadV2/xyp-gpib.kicad_sch (KiCad schematic)
At the start: 25 parts, among them J1 USB_C_Receptacle_USB2.0, SW1 SW_Push, U1 ATmega32U4-MU, Y1 CX2016DB16000D0WZRC1

Commit message: commit
Connections:
- net GND: now also GPIB1.MH1
- net Db+: now reaches R2.1, U1.3 (D-)
- net Db-: now reaches R3.1, U1.4 (D+)
- net D+ renamed Da+
- net D- renamed Da-
- no-connect marks 0 -> 7
Other:
- note added: "GPIB CONNECTOR"
- note added: "JLC04161H-3313 Stackup"
- company: (none) -> xyphro
- title: (none) -> UsbGpib
- moved on the sheet: C1, C2, C3, C4, C5, C6, C7, D1, D2, FID1, FID2, GPIB1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
